Commit message: 260904-1112

File: joyarm_code/joyarm_core/robot_model/joyarm_dm/urdf/00-arm-rs_asm-v3.urdf (robot description, URDF)
Before this commit: robot 00-arm-rs_asm-v3, 10 links, 9 joints
Links:
- removed link base_link
- added link link_base, mass 1.1774; collision mesh filename=../meshes/link_base.STL; visual mesh filename=../meshes/link_base.STL
Joints:
- joint joint1: parent base_link -> link_base

File: joyarm_code/joyarm_core/robot_model/joyarm_dm_fixend/urdf/joyarm_dm_fixend.urdf (robot description, URDF)
Before this commit: robot joyarm_dm_fixend, 8 links, 7 joints
Links:
- removed link base_link
- removed link end_link
- added link link_base, mass 0.83660000; collision mesh filename=../meshes/link_base.STL; visual mesh filename=../meshes/link_base.STL
- added link link_end, mass 0.4500000; collision mesh filename=../meshes/link_end.STL; visual mesh filename=../meshes/link_end.STL
Joints:
- joint end_joint: child end_link -> link_end
- joint joint1: parent base_link -> link_base
