Commit message: 260914-1812

File: joyarm_code/joyarm_core/robot_model/joyarm_dm/urdf/joyarm_dm.urdf (robot description, URDF)
Before this commit: robot 00-arm-rs_asm-v3, 10 links, 9 joints
Links:
- removed link gripper_end
- removed link gripper_left
- removed link gripper_right
- added link frame_end_fingertip
- added link frame_end_tcp
- added link link_end, mass 0.432; collision mesh filename=../meshes/link_end.STL; visual mesh filename=../meshes/link_end.STL
- added link link_end1, mass 0.023; collision mesh filename=../meshes/link_end1.STL; visual mesh filename=../meshes/link_end1.STL
- added link link_end_finger1, mass 0.085; collision mesh filename=../meshes/link_end_finger1.STL; visual mesh filename=../meshes/link_end_finger1.STL
- added link link_end_finger2, mass 0.085; collision mesh filename=../meshes/link_end_finger2.STL; visual mesh filename=../meshes/link_end_finger2.STL
- link link1: mass 0.4655 -> 0.217
- link link2: mass 1.552 -> 1.196; geometry collision mesh filename=../meshes/link2.STL; visual mesh filename=../meshes/link2.STL
- link link3: mass 1.252 -> 0.799; geometry collision mesh filename=../meshes/link3.STL; visual mesh filename=../meshes/link3.STL
- link link4: mass 0.46 -> 0.473; geometry collision mesh filename=../meshes/link4.STL; visual mesh filename=../meshes/link4.STL
- link link5: mass 0.20120457182895 -> 0.375; geometry collision mesh filename=../meshes/link5.STL; visual mesh filename=../meshes/link5.STL
- link link6: mass 0.1 -> 0.070
- link link_base: mass 1.1774 -> 0.808
Joints:
- removed joint j_gripper_end
- removed joint joint_left
- removed joint joint_right
- added joint joint_end: type fixed, parent link6, child link_end, origin xyz=0 0 0.032692 rpy=1.5708 -1.5708 0, axis 0 0 0
- added joint joint_end1: type revolute, parent link_end, child link_end1, origin xyz=0.0485 0 0 rpy=0 0 0, axis 1 0 0, limit lower=-5.49 upper=0 effort=7 velocity=20
- added joint joint_end_pris1: type prismatic, parent link_end, child link_end_finger1, origin xyz=0.0859 2.7531E-05 -1.3031E-05 rpy=0 0 0, axis 0 1 -0.00014746, limit lower=-0.04625 upper=0 effort=7 velocity=0.08, mimic joint=joint_end1 multiplier=0.00842 offset=0
- added joint joint_end_pris2: type prismatic, parent link_end, child link_end_finger2, origin xyz=0.0859 -2.7531E-05 1.3031E-05 rpy=0 0 0, axis 0 -1 0.00014746, limit lower=-0.04625 upper=0 effort=7 velocity=0.08, mimic joint=joint_end1 multiplier=0.00842 offset=0
- added joint joint_frame_end_fingertip: type fixed, parent link_end, child frame_end_fingertip, origin xyz=0.15071 0 -0.00001 rpy=0 0 0
- added joint joint_frame_end_tcp: type fixed, parent link_end, child frame_end_tcp, origin xyz=0.12510 0 0 rpy=0 0 0
- joint joint1: axis 0 0 -1 -> 0 0 1; limit lower=-2.8 upper=2.8 effort=36 velocity=50 -> lower=-2.8 upper=2.8 effort=27 velocity=5; origin xyz=-0.00034283 -0.00098683 0.075 rpy=0 0 0 -> xyz=0 0 0.1402 rpy=0 0 0
- joint joint2: limit lower=0 upper=3.14 effort=36 velocity=50 -> lower=0 upper=3.14 effort=27 velocity=5; origin xyz=0.020343 0.027237 0.07 rpy=-1.5708 0 0 -> xyz=0.02 0 0 rpy=1.5708 0 3.1416
- joint joint3: axis 0 0 -1 -> 0 0 1; limit lower=0 upper=3.14 effort=36 velocity=50 -> lower=-3.14 upper=0 effort=27 velocity=5; origin xyz=-0.236 0 0 rpy=0 0 0 -> xyz=0.264 0 0 rpy=0 0 2.9226
- joint joint4: axis 0 0 -1 -> 0 0 1; limit lower=-1.57 upper=1.57 effort=14 velocity=40 -> lower=-1.57 upper=1.57 effort=7 velocity=20; origin xyz=0.228 -0.072746 0.0045 rpy=0 0 0 -> xyz=0.24854 0 0 rpy=0 -0.030795 0.21913
- joint joint5: axis 0 0 -1 -> 0 0 1; limit lower=-1.57 upper=1.57 effort=14 velocity=40 -> lower=-1.57 upper=1.57 effort=7 velocity=20; origin xyz=0.087 -0.048 -0.03075 rpy=-1.5708 0 0 -> xyz=0.078283 0.0024911 -0.0016418 rpy=1.571 1.54 -3.1416
- joint joint6: axis 0 0 -1 -> 0 0 1; limit lower=-3.14 upper=3.14 effort=14 velocity=40 -> lower=-3.14 upper=3.14 effort=7 velocity=20; origin xyz=0.0365 0 0.048 rpy=0 1.5708 0 -> xyz=0.00076939 -1.1537E-05 0 rpy=1.5707 0 0

Commit message: 260915-1115

File: joyarm_code/joyarm_core/robot_model/joyarm_dm/urdf/joyarm_dm.urdf (robot description, URDF)
Before this commit: robot joyarm_dm, 13 links, 12 joints
Joints:
- joint joint2: axis 0 0 1 -> 0 0 -1; limit lower=0 upper=3.14 effort=27 velocity=5 -> lower=-3.14 upper=0 effort=27 velocity=5

Commit message: 260915-1142

File: joyarm_code/joyarm_core/robot_model/joyarm_dm/urdf/joyarm_dm.urdf (robot description, URDF)
Before this commit: robot joyarm_dm, 13 links, 12 joints
Joints:
- joint joint2: axis 0 0 -1 -> 0 0 1; origin xyz=0.02 0 0 rpy=1.5708 0 3.1416 -> xyz=0.02 0 0 rpy=-1.570792653589793 0 3.1416
- joint joint3: origin xyz=0.264 0 0 rpy=0 0 2.9226 -> xyz=0.264 0 0 rpy=3.141592653589793 0 -2.9226

Commit message: 260919-1443

File: joyarm_code/joyarm_core/robot_model/joyarm_dm/urdf/joyarm_dm.urdf (robot description, URDF)
Before this commit: robot joyarm_dm, 13 links, 12 joints
Links:
- removed link link_base
- removed link link_end
- removed link link_end_finger1
- removed link link_end_finger2
- added link link0, mass 0.808; collision mesh filename=../meshes/link0.STL; visual mesh filename=../meshes/link0.STL
- added link link_end0, mass 0.432; collision mesh filename=../meshes/link_end0.STL; visual mesh filename=../meshes/link_end0.STL
- added link link_end_fingerleft, mass 0.085; collision mesh filename=../meshes/link_end_fingerleft.STL; visual mesh filename=../meshes/link_end_fingerleft.STL
- added link link_end_fingerright, mass 0.085; collision mesh filename=../meshes/link_end_fingerright.STL; visual mesh filename=../meshes/link_end_fingerright.STL
Joints:
- removed joint joint_end
- removed joint joint_end_pris1
- removed joint joint_end_pris2
- added joint joint_end0: type fixed, parent link6, child link_end0, origin xyz=0 0 0.032692 rpy=1.5708 -1.5708 0
- added joint joint_end_fingerleft: type prismatic, parent link_end0, child link_end_fingerleft, origin xyz=0.0859 -2.7531E-05 1.3031E-05 rpy=0 0 0, axis 0 -1 0.00014746, limit lower=-0.04625 upper=0 effort=178.15 velocity=0.06736, mimic joint=joint_end1 multiplier=0.00842 offset=0
- added joint joint_end_fingerright: type prismatic, parent link_end0, child link_end_fingerright, origin xyz=0.0859 2.7531E-05 -1.3031E-05 rpy=0 0 0, axis 0 1 -0.00014746, limit lower=-0.04625 upper=0 effort=178.15 velocity=0.06736, mimic joint=joint_end1 multiplier=0.00842 offset=0
- joint joint1: limit lower=-2.8 upper=2.8 effort=27 velocity=5 -> lower=-2.8 upper=2.8 effort=30 velocity=5; parent link_base -> link0
- joint joint2: limit lower=-3.14 upper=0 effort=27 velocity=5 -> lower=-3.14 upper=0 effort=30 velocity=5
- joint joint3: limit lower=-3.14 upper=0 effort=27 velocity=5 -> lower=-3.14 upper=0 effort=30 velocity=5
- joint joint4: limit lower=-1.57 upper=1.57 effort=7 velocity=20 -> lower=-1.57 upper=1.57 effort=9 velocity=8
- joint joint5: limit lower=-1.57 upper=1.57 effort=7 velocity=20 -> lower=-1.57 upper=1.57 effort=9 velocity=8
- joint joint6: limit lower=-3.14 upper=3.14 effort=7 velocity=20 -> lower=-3.14 upper=3.14 effort=9 velocity=8
- joint joint_end1: limit lower=-5.49 upper=0 effort=7 velocity=20 -> lower=-5.49 upper=0 effort=1.5 velocity=8; parent link_end -> link_end0
- joint joint_frame_end_fingertip: parent link_end -> link_end0
- joint joint_frame_end_tcp: parent link_end -> link_end0

Commit message: feat(kinematics): 增加 MDH 正解与解析逆解

File: joyarm_code/joyarm_core/robot_model/joyarm_dm/urdf/joyarm_dm.urdf (robot description, URDF)
Before this commit: robot joyarm_dm, 13 links, 12 joints
Joints:
- joint joint2: origin xyz=0.02 0 0 rpy=-1.570792653589793 0 3.1416 -> xyz=0.02 0 0 rpy=-1.5707963267948966 0 3.141592653589793
- joint joint4: origin xyz=0.24854 0 0 rpy=0 -0.030795 0.21913 -> xyz=0.24854 0 0 rpy=0 0 0.21913
- joint joint6: origin xyz=0.00076939 -1.1537E-05 0 rpy=1.5707 0 0 -> xyz=0 0 0 rpy=1.5707963267948966 0 0
